Commit message: Began implementing micro module URDF model.

File: urdf/micro_module.urdf (robot description, URDF)
Before this commit: robot micro_module, 10 links, 0 joints
Links:
- removed link control box
- removed link distal_module_3
- removed link proximal_module_3
- added link control_box; visual box size=0.154 0.114 0.052
- added link proximal_base; visual mesh filename=package://ls_thesis/meshes/proximal_base.stl scale=0.001 0.001 0.001
- added link tube_base; visual mesh filename=package://ls_thesis/meshes/tube_base.stl scale=0.001 0.001 0.001
- link distal_module_1: geometry visual mesh filename=package://ls_thesis/meshes/distal_module.stl scale=0.001 0.001 0.001
- link distal_module_2: geometry visual mesh filename=package://ls_thesis/meshes/distal_module.stl scale=0.001 0.001 0.001
- link end_effector: geometry visual mesh filename=package://ls_thesis/meshes/distal_module.stl scale=0.001 0.001 0.001
- link pd_adaptor_module: geometry visual mesh filename=package://ls_thesis/meshes/pd_adaptor_module.stl scale=0.001 0.001 0.001
- link proximal_module_1: geometry visual mesh filename=package://ls_thesis/meshes/proximal_module.stl scale=0.001 0.001 0.001
- link proximal_module_2: geometry visual mesh filename=package://ls_thesis/meshes/proximal_module.stl scale=0.001 0.001 0.001
- link steel_tube: geometry visual cylinder length=0.25 radius=0.002
Joints:
- added joint link_control_box:tube_base: type fixed, parent control_box, child tube_base, origin xyz=0 0 0 rpy=0 0 0
- added joint link_distal_module_1:distal_module_2: type fixed, parent distal_module_1, child distal_module_2, origin xyz=0 0 0 rpy=0 0 0
- added joint link_distal_module_2:end_effector: type fixed, parent distal_module_2, child end_effector, origin xyz=0 0 0 rpy=0 0 0
- added joint link_pd_adaptor_module:distal_module_1: type fixed, parent pd_adaptor_module, child distal_module_1, origin xyz=0 0 0 rpy=0 0 0
- added joint link_proximal_base:proximal_module_1: type fixed, parent proximal_base, child proximal_module_1, origin xyz=0 0 0 rpy=0 0 0
- added joint link_proximal_module_1:proximal_module_2: type fixed, parent proximal_module_1, child proximal_module_2, origin xyz=0 0 0 rpy=0 0 0
- added joint link_proximal_module_2:pd_adaptor_module: type fixed, parent proximal_module_2, child pd_adaptor_module, origin xyz=0 0 0 rpy=0 0 0
- added joint link_steel_tube:proximal_base: type fixed, parent steel_tube, child proximal_base, origin xyz=0 0 0 rpy=0 0 0
- added joint link_tube_base:steel_tube: type fixed, parent tube_base, child steel_tube, origin xyz=0 0 0 rpy=0 0 0

Commit message: Complete link positioning of  micro module URDF.

File: urdf/micro_module.urdf (robot description, URDF)
Before this commit: robot micro_module, 10 links, 9 joints
Links:
- link end_effector: geometry visual mesh filename=package://ls_thesis/meshes/end_effector.stl scale=0.001 0.001 0.001
Joints:
- joint link_distal_module_1:distal_module_2: axis (none) -> 0 0 1; type fixed -> revolute
- joint link_distal_module_2:end_effector: axis (none) -> 0 0 1; type fixed -> revolute
- joint link_pd_adaptor_module:distal_module_1: axis (none) -> 0 0 1; type fixed -> revolute
- joint link_proximal_base:proximal_module_1: axis (none) -> 0 0 1; type fixed -> revolute
- joint link_proximal_module_1:proximal_module_2: axis (none) -> 0 0 1; type fixed -> revolute
- joint link_proximal_module_2:pd_adaptor_module: axis (none) -> 0 0 1; type fixed -> revolute

Commit message: Added revolute joint limits.

File: urdf/micro_module.urdf (robot description, URDF)
Before this commit: robot micro_module, 10 links, 9 joints
Joints:
- joint link_distal_module_1:distal_module_2: limit (none) -> lower=0.0 upper=0.548 effort=1000.0 velocity=0.5
- joint link_distal_module_2:end_effector: limit (none) -> lower=0.0 upper=0.548 effort=1000.0 velocity=0.5
- joint link_pd_adaptor_module:distal_module_1: limit (none) -> lower=0.0 upper=0.548 effort=1000.0 velocity=0.5
- joint link_proximal_base:proximal_module_1: limit (none) -> lower=0.0 upper=0.548 effort=1000.0 velocity=0.5
- joint link_proximal_module_1:proximal_module_2: limit (none) -> lower=0.0 upper=0.548 effort=1000.0 velocity=0.5
- joint link_proximal_module_2:pd_adaptor_module: limit (none) -> lower=0.0 upper=0.548 effort=1000.0 velocity=0.5

Commit message: Corrected link and joint origins.

File: urdf/micro_module.urdf (robot description, URDF)
Before this commit: robot micro_module, 10 links, 9 joints
Joints:
- removed joint link_control_box:tube_base
- removed joint link_distal_module_1:distal_module_2
- removed joint link_distal_module_2:end_effector
- removed joint link_pd_adaptor_module:distal_module_1
- removed joint link_proximal_base:proximal_module_1
- removed joint link_proximal_module_1:proximal_module_2
- removed joint link_proximal_module_2:pd_adaptor_module
- removed joint link_steel_tube:proximal_base
- removed joint link_tube_base:steel_tube
- added joint joint_control_box:tube_base: type fixed, parent control_box, child tube_base, origin xyz=0 0 0 rpy=0 0 0
- added joint joint_distal_module_1:distal_module_2: type revolute, parent distal_module_1, child distal_module_2, origin xyz=-0.0027 0 0 rpy=0 0 0, axis 0 1 0, limit lower=-0.6 upper=0.6 effort=1000.0 velocity=0.5
- added joint joint_distal_module_2:end_effector: type revolute, parent distal_module_2, child end_effector, origin xyz=-0.00275 0 0 rpy=0 0 0, axis 0 0 1, limit lower=-0.6 upper=0.6 effort=1000.0 velocity=0.5
- added joint joint_pd_adaptor_module:distal_module_1: type revolute, parent pd_adaptor_module, child distal_module_1, origin xyz=-0.00251 0 0 rpy=0.7854 0 0, axis 0 0 1, limit lower=-0.6 upper=0.6 effort=1000.0 velocity=0.5
- added joint joint_proximal_base:proximal_module_1: type revolute, parent proximal_base, child proximal_module_1, origin xyz=0 0.3120 0 rpy=-0.78540 0 -1.570796, axis 0 0 1, limit lower=-0.15 upper=0.15 effort=1000.0 velocity=0.5
- added joint joint_proximal_module_1:proximal_module_2: type revolute, parent proximal_module_1, child proximal_module_2, origin xyz=-0.0014 0 0 rpy=1.570796 0 0, axis 0 0 1, limit lower=-0.15 upper=0.15 effort=1000.0 velocity=0.5
- added joint joint_proximal_module_2:pd_adaptor_module: type revolute, parent proximal_module_2, child pd_adaptor_module, origin xyz=-0.0014 0 0 rpy=1.570796 0 0, axis 0 0 1, limit lower=-0.15 upper=0.15 effort=1000.0 velocity=0.5
- added joint joint_steel_tube:proximal_base: type fixed, parent steel_tube, child proximal_base, origin xyz=0 0 0 rpy=0 0 0
- added joint joint_tube_base:steel_tube: type fixed, parent tube_base, child steel_tube, origin xyz=0 0 0 rpy=0 0 0
